Commit message: Second Commit

File: src/mobile_platform_descpription/urdf/mobile_platform_description_v1.xacro (robot description, xacro)
@@ -414,9 +414,11 @@
     <collision>
       <origin
-        xyz="0 0 0"
-        rpy="0 0 0" />
-      <geometry>
-        <mesh
-          filename="package://dualarm_config/meshes/mani1_link2.STL" />
+        xyz="0 0 .09"
+        rpy="0 0 0" />
+      <geometry>
+<!--
+        <mesh
+          filename="package://dualarm_config/meshes/mani1_link2.STL" /> -->
+        <box size=".15 .16 .19"/>
       </geometry>
     </collision>
@@ -475,9 +477,10 @@
     <collision>
       <origin
-        xyz="0 0 0"
-        rpy="0 0 0" />
-      <geometry>
-        <mesh
-          filename="package://dualarm_config/meshes/mani1_link3.STL" />
+        xyz="0 -0.13 0"
+        rpy="0 0 0" />
+      <geometry>
+        <!--<mesh
+          filename="package://dualarm_config/meshes/mani1_link3.STL" />-->
+        <box size=".12 .24 .12"/>
       </geometry>
     </collision>
@@ -536,9 +539,10 @@
     <collision>
       <origin
-        xyz="0 0 0"
-        rpy="0 0 0" />
-      <geometry>
-        <mesh
-          filename="package://dualarm_config/meshes/mani1_link4.STL" />
+        xyz="0 0 .09"
+        rpy="0 0 0" />
+      <geometry>
+        <!--<mesh
+          filename="package://dualarm_config/meshes/mani1_link4.STL" />-->
+        <box size=".1 .1 .18"/>
       </geometry>
     </collision>
@@ -597,9 +601,10 @@
     <collision>
       <origin
-        xyz="0 0 0"
-        rpy="0 0 0" />
-      <geometry>
-        <mesh
-          filename="package://dualarm_config/meshes/mani1_link5.STL" />
+        xyz="0 -0.11 0"
+        rpy="0 0 0" />
+      <geometry>
+        <!--<mesh
+          filename="package://dualarm_config/meshes/mani1_link5.STL" />-->
+        <box size=".09 .20 .09"/>
       </geometry>
     </collision>
@@ -658,9 +663,10 @@
     <collision>
       <origin
-        xyz="0 0 0"
-        rpy="0 0 0" />
-      <geometry>
-        <mesh
-          filename="package://dualarm_config/meshes/mani1_link6.STL" />
+        xyz="0 0 .09"
+        rpy="0 0 0" />
+      <geometry>
+        <!--<mesh
+          filename="package://dualarm_config/meshes/mani1_link6.STL" /> -->
+	<box size=".09 .08 .18"/>
       </geometry>
     </collision>
@@ -719,9 +725,10 @@
     <collision>
       <origin
-        xyz="0 0 0"
-        rpy="0 0 0" />
-      <geometry>
-        <mesh
-          filename="package://dualarm_config/meshes/mani1_link7.STL" />
+        xyz="0 -0.09 0"
+        rpy="0 0 0" />
+      <geometry>
+        <!--<mesh
+          filename="package://dualarm_config/meshes/mani1_link7.STL" />-->
+        <box size=".08 .18 .08"/>
       </geometry>
     </collision>
@@ -780,9 +787,10 @@
     <collision>
       <origin
-        xyz="0 0 0"
-        rpy="0 0 0" />
-      <geometry>
-        <mesh
-          filename="package://dualarm_config/meshes/mani1_eef.STL" />
+        xyz="0 0 0.08"
+        rpy="0 0 0" />
+      <geometry>
+        <!--<mesh
+          filename="package://dualarm_config/meshes/mani1_eef.STL" />-->
+	<box size=".16 .18 .16"/>
       </geometry>
     </collision>
@@ -809,4 +817,6 @@
       velocity="0.8" />
   </joint>
+<!-- distance between two manipulator is 46cm (=0.46/2 =0.23) -->
+<!-- height between base origin to manipulator base is 11.2cm (=0.112) -->
   <joint
     name="base_joint_right"
@@ -822,4 +832,5 @@
       xyz="0 0 0" />
   </joint>
+<!-- Mani2 base -->
   <link
     name="mani2_base">
@@ -1237,9 +1248,10 @@
     <collision>
       <origin
-        xyz="0 0 0"
-        rpy="0 0 0" />
-      <geometry>
-        <mesh
-          filename="package://dualarm_config/meshes/mani2_link7.STL" />
+        xyz="0 -0.03 0"
+        rpy="0 0 0" />
+      <geometry>
+        <!--<mesh
+          filename="package://dualarm_config/meshes/mani2_link7.STL" />-->
+	<box size=".08 .13 .16"/>
       </geometry>
     </collision>
@@ -1321,5 +1333,5 @@
       velocity="0.8" />
   </joint>
-<!--transmissions-->
+<!-- Transmissions for ROS Control -->
   <transmission name="left_tran1">
     <type>transmission_interface/SimpleTransmission</type>
@@ -1462,4 +1474,5 @@
     </actuator>
   </transmission>
+  <!-- ros_control plugin -->
   <gazebo>
     <plugin filename="libgazebo_ros_control.so" name="gazebo_ros_control">

File: src/mservo_manipulator_control-main/dualarm_config/urdf/dualarm.urdf (robot description, URDF)
Before this commit: robot dualarm, 19 links, 18 joints
Links:
- added link camera; collision box size=.15 .7 .05; visual box size=.15 .7 .05
- added link dummy_link
- added link lidar1; collision box size=.08 .08 .06; visual box size=.08 .08 .06
- added link table; collision box size=.72 .6 .03; visual box size=.72 .6 .03
- link mani1_eff: geometry collision box size=.16 .18 .16; visual mesh filename=package://dualarm_config/meshes/mani1_eef.STL
- link mani1_link2: geometry collision box size=.15 .16 .19; visual mesh filename=package://dualarm_config/meshes/mani1_link2.STL
- link mani1_link3: geometry collision box size=.12 .24 .12; visual mesh filename=package://dualarm_config/meshes/mani1_link3.STL
- link mani1_link4: geometry collision box size=.1 .1 .18; visual mesh filename=package://dualarm_config/meshes/mani1_link4.STL
- link mani1_link5: geometry collision box size=.09 .20 .09; visual mesh filename=package://dualarm_config/meshes/mani1_link5.STL
- link mani1_link6: geometry collision box size=.09 .08 .18; visual mesh filename=package://dualarm_config/meshes/mani1_link6.STL
- link mani1_link7: geometry collision box size=.08 .18 .08; visual mesh filename=package://dualarm_config/meshes/mani1_link7.STL
- link mani2_link7: geometry collision box size=.08 .13 .16; visual mesh filename=package://dualarm_config/meshes/mani2_link7.STL
Joints:
- added joint camera_joint: type fixed, parent base_link, child camera, origin xyz=0 -0.85 0.890 rpy=0 0 0, axis 0 0 0
- added joint dummy_joint: type fixed, parent dummy_link, child base_link, origin xyz=0 0 0 rpy=0 0 0
- added joint lidar1_joint: type fixed, parent base_link, child lidar1, origin xyz=-0.28 -0.175 0.40 rpy=0 0 0, axis 0 0 0
- added joint table_joint: type fixed, parent base_link, child table, origin xyz=0 -0.45 0.2 rpy=0 0 0, axis 0 0 0
