Commit message: Branch First Commit

File: src/mservo_manipulator_control-main/dualarm_config/urdf/dualarm.urdf (robot description, URDF)
Before this commit: robot dualarm, 23 links, 22 joints
Links:
- removed link camera
- removed link lidar1
- removed link table
- link dummy_link: mass None -> 10000
Joints:
- removed joint camera_joint
- removed joint lidar1_joint
- removed joint table_joint
- joint dummy_joint: type fixed -> planar

Commit message: Add Platform Control

File: src/mservo_manipulator_control-main/dualarm_config/urdf/dualarm.urdf (robot description, URDF)
Before this commit: robot dualarm, 20 links, 19 joints
Links:
- added link dummy_link_1, mass 1
- added link dummy_link_2, mass 1
- added link world
- link dummy_link: mass 10000 -> 1
Joints:
- added joint dummy_joint_1: type prismatic, parent dummy_link_1, child dummy_link_2, origin xyz=0 0 0 rpy=0 0 1.5708, limit lower=-12.74 upper=12.74 effort=100 velocity=0.8
- added joint dummy_joint_2: type revolute, parent dummy_link_2, child base_link, origin xyz=0 0 0 rpy=0 0 0, axis 0 0 1, limit lower=-2.74 upper=2.74 effort=100 velocity=0.8
- added joint dummy_joint_x: type fixed, parent world, child dummy_link, origin xyz=0 0 0 rpy=0 0 0
- joint dummy_joint: child base_link -> dummy_link_1; limit (none) -> lower=-12.74 upper=12.74 effort=100 velocity=0.8; type planar -> prismatic

Commit message: First Commit

File: src/mservo_manipulator_control-main/dualarm_config/urdf/dualarm.urdf (robot description, URDF)
Before this commit: robot dualarm, 23 links, 22 joints
Links:
- removed link dummy_link_1
- removed link dummy_link_2
- added link dummy_link_l1, mass 10
- added link dummy_link_l2, mass 10
Joints:
- removed joint dummy_joint
- removed joint dummy_joint_1
- removed joint dummy_joint_2
- removed joint dummy_joint_x
- added joint dummy_joint_l1: type prismatic, parent dummy_link, child dummy_link_l1, origin xyz=0 0 0 rpy=0 0 1.5708, limit lower=-12.74 upper=12.74 effort=100 velocity=0.8
- added joint dummy_joint_l2: type prismatic, parent dummy_link_l1, child dummy_link_l2, origin xyz=0 0 0 rpy=0 0 1.5708, limit lower=-12.74 upper=12.74 effort=100 velocity=0.8
- added joint dummy_joint_l3: type revolute, parent dummy_link_l2, child base_link, origin xyz=0 0 0 rpy=0 0 0, axis 0 0 1, limit lower=-12.74 upper=12.74 effort=100 velocity=0.8
- added joint world_joint: type fixed, parent world, child dummy_link, origin xyz=0 0 0 rpy=0 0 0
